File: docs/schematics/aac/Shield.kicad_pcb (KiCad board)
At the start: 2 copper layers, 71 parts, among them J1 CONN_LED_ORG, J10 But_4, J11 But_5, J12 Camera, J16 Conn_01x22_Female, J2 CONN_LED_RED, J3 HAT, J5 Actuator, J6 RS232, J6 THD-02-R, J7 But_1, J8 But_2, J8 THD-20-R, J9 But_3, J9 THD-02-R, U1 TXU0202, U2 TJA1050, U3 MCP2515-xSO, U5 MAX3232

Commit message: Pushing final schematic and PCB.
Parts:
- removed the C10 at (24.8, 102.4)
- removed the C11 at (24.8, 105.4)
- removed the C12 at (24.8, 108.4)
- removed the C14 at (29.2, 96.4)
- removed the C15 at (29.2, 99.4)
- removed the C9 at (24.8, 99.4)
- removed H5: MountingHole, MountingHole:MountingHole_2.7mm_M2.5
- removed the J16 at (89.5, 65.2)
- removed the J16 at (82.9, 83.6)
- removed the J16 at (125.5, 65.2)
- removed the J5 at (34.6, 40.2)
- removed the J6 at (21.2, 40.2)
- removed the J6 at (119.4, 93.4)
- removed the J8 at (86.3, 99.0)
- removed the J8 at (39.6, 65.2)
- removed the J9 at (44.3, 65.2)
- removed the J9 at (138.2, 102.5)
- removed the R12 at (51.7, 77.0)
- removed the R6 at (38.0, 93.3)
- removed the R8 at (38.0, 99.2)
- removed REF**: SO-16_5.3x10.2mm_P1.27mm, Package_SO:SO-16_5.3x10.2mm_P1.27mm
- removed REF**: SO-16_3.9x9.9mm_P1.27mm, Package_SO:SO-16_3.9x9.9mm_P1.27mm
- removed REF** (x2): TE_1-84952-5_1x15-1MP_P1.0mm_Horizontal, Connector_FFC-FPC:TE_1-84952-5_1x15-1MP_P1.0mm_Horizontal
- removed REF**: Hirose_FH12-40S-0.5SH_1x40-1MP_P0.50mm_Horizontal, Connector_FFC-FPC:Hirose_FH12-40S-0.5SH_1x40-1MP_P0.50mm_Horizontal
- removed the U3 at (47.6, 125.4)
- added C19: 100n, Capacitor_SMD:C_0805_2012Metric, F.Cu at (105.0, 63.0)
- added C20: 100n, Capacitor_SMD:C_0805_2012Metric, F.Cu at (88.9, 104.0)
- added C21: 100n, Capacitor_SMD:C_0805_2012Metric, F.Cu at (95.1, 108.8)
- added C22: 100n, Capacitor_SMD:C_0805_2012Metric, F.Cu at (95.1, 113.3)
- added C23: 100n, Capacitor_SMD:C_0805_2012Metric, F.Cu at (95.1, 117.8)
- added C24: 100n, Capacitor_SMD:C_0805_2012Metric, F.Cu at (95.1, 122.3)
- added C25: 100n, Capacitor_SMD:C_0805_2012Metric, F.Cu at (95.1, 126.8)
- added C26: 100n, Capacitor_SMD:C_0805_2012Metric, F.Cu at (95.1, 131.3)
- added C27: 100n, Capacitor_SMD:C_0805_2012Metric, F.Cu at (95.1, 135.8)
- added C6: 100n, Capacitor_SMD:C_0805_2012Metric, F.Cu at (111.0, 119.5)
- added C7: 100n, Capacitor_SMD:C_0805_2012Metric, F.Cu at (111.0, 111.5)
- added G***: LOGO, LOGO, F.Cu at (111.2, 135.5)
- added J12: Berry_CAM1, Connector_FFC-FPC:Hirose_FH12-22S-0.5SH_1x22-1MP_P0.50mm_Horizontal, B.Cu at (89.5, 65.2)
- added J13: But_1, Connector_PinHeader_2.54mm:PinHeader_2x01_P2.54mm_Horizontal, F.Cu at (90.4, 109.0)
- added J14: But_2, Connector_PinHeader_2.54mm:PinHeader_2x01_P2.54mm_Horizontal, F.Cu at (90.4, 113.3)
- added J15: But_3, Connector_PinHeader_2.54mm:PinHeader_2x01_P2.54mm_Horizontal, F.Cu at (90.4, 117.8)
- added J16: But_4, Connector_PinHeader_2.54mm:PinHeader_2x01_P2.54mm_Horizontal, F.Cu at (90.4, 122.3)
- added J17: But_5, Connector_PinHeader_2.54mm:PinHeader_2x01_P2.54mm_Horizontal, F.Cu at (90.4, 126.8)
- added J18: But_6, Connector_PinHeader_2.54mm:PinHeader_2x01_P2.54mm_Horizontal, F.Cu at (90.4, 131.3)
- added J19: But_7, Connector_PinHeader_2.54mm:PinHeader_2x01_P2.54mm_Horizontal, F.Cu at (90.4, 135.8)
- added J20: Berry_DISP1, Connector_FFC-FPC:Hirose_FH12-22S-0.5SH_1x22-1MP_P0.50mm_Horizontal, B.Cu at (125.5, 65.2)
- added J21: Display, Connector_FFC-FPC:Hirose_FH12-40S-0.5SH_1x40-1MP_P0.50mm_Horizontal, F.Cu at (122.0, 65.4)
- added J3: CONN_LED_RED, Connector_PinHeader_2.54mm:PinHeader_2x01_P2.54mm_Horizontal, F.Cu at (130.3, 118.5)
- added J4: CONN_LED_AUX, Connector_PinHeader_2.54mm:PinHeader_2x01_P2.54mm_Horizontal, F.Cu at (130.3, 123.0)
- added J6: Actuator, Connector_PinHeader_2.54mm:PinHeader_2x03_P2.54mm_Vertical, F.Cu at (116.3, 122.7)
- added J8: RS232, Connector_PinHeader_2.54mm:PinHeader_1x06_P2.54mm_Horizontal, F.Cu at (130.2, 80.0)
- added JP1: Jumper_2_Open, Jumper:SolderJumper-2_P1.3mm_Open_RoundedPad1.0x1.5mm, F.Cu at (121.7, 72.6)
- added JP2: Jumper_2_Open, Jumper:SolderJumper-2_P1.3mm_Open_RoundedPad1.0x1.5mm, F.Cu at (121.7, 75.2)
- added R13: 10K, Resistor_SMD:R_0805_2012Metric, F.Cu at (98.1, 108.8)
- added R14: 10K, Resistor_SMD:R_0805_2012Metric, F.Cu at (98.1, 113.3)
- added R15: 10K, Resistor_SMD:R_0805_2012Metric, F.Cu at (98.1, 117.8)
- added R16: 10K, Resistor_SMD:R_0805_2012Metric, F.Cu at (98.1, 122.3)
- added R17: 10K, Resistor_SMD:R_0805_2012Metric, F.Cu at (98.1, 126.8)
- added R18: 10K, Resistor_SMD:R_0805_2012Metric, F.Cu at (98.1, 131.3)
- added R19: 10K, Resistor_SMD:R_0805_2012Metric, F.Cu at (98.1, 135.8)
- added R3: 140, Resistor_SMD:R_0805_2012Metric, F.Cu at (125.5, 123.0)
- added R4: 140, Resistor_SMD:R_0805_2012Metric, F.Cu at (131.8, 126.5)
- added SW1: SW_Clutch, Connector_PinHeader_2.54mm:PinHeader_2x01_P2.54mm_Horizontal, F.Cu at (130.3, 108.5)
- added SW2: SW_Brake, Connector_PinHeader_2.54mm:PinHeader_2x01_P2.54mm_Horizontal, F.Cu at (130.3, 104.0)
- C13: value 100n -> 2.2uF
- J1: value CONN_LED_ORG -> 12V; footprint Connector_PinHeader_2.54mm:PinHeader_1x02_P2.54mm_Vertical -> Connector_PinHeader_2.54mm:PinHeader_1x02_P2.54mm_Horizontal
- J10: value But_4 -> Camera; footprint Connector_PinHeader_2.54mm:PinHeader_1x02_P2.54mm_Vertical -> Connector_FFC-FPC:TE_1-84952-5_1x15-1MP_P1.0mm_Horizontal
- J11: value But_5 -> Berry_CAM0; footprint Connector_PinHeader_2.54mm:PinHeader_1x02_P2.54mm_Vertical -> Connector_FFC-FPC:Hirose_FH12-22S-0.5SH_1x22-1MP_P0.50mm_Horizontal; moved to B.Cu
- J2: value CONN_LED_RED -> CONN_LED_ORG; footprint Connector_PinHeader_2.54mm:PinHeader_1x02_P2.54mm_Vertical -> Connector_PinHeader_2.54mm:PinHeader_2x01_P2.54mm_Horizontal
- J5: renamed from J3; moved to B.Cu
- J7: value But_1 -> CAN_Module; footprint Connector_PinHeader_2.54mm:PinHeader_1x02_P2.54mm_Vertical -> Connector_PinHeader_2.54mm:PinHeader_1x07_P2.54mm_Vertical
- L1: value 47 uH -> 330 uH; footprint Inductor_SMD:L_7.3x7.3_H4.5 -> Inductor_SMD:L_SigTra_SC3316F
- R10: value 10k -> 5.1K
- R11: value 10K -> PT15LV 25K; footprint Resistor_SMD:R_0805_2012Metric -> Potentiometer_THT:Potentiometer_ACP_CA14V-15_Vertical
- R20: renamed from R14; value 10k -> 10K
- R5: renamed from R3; value 10k -> 10K
- R6: renamed from R4; value 10k -> 10K
- R7, R9: value 10k -> 1K
- U2: value TJA1050 -> TPS92511DDA; footprint Package_SO:SOIC-8_3.9x4.9mm_P1.27mm -> Package_SO:SOIC-8-1EP_3.9x4.9mm_P1.27mm_EP2.29x3mm_ThermalVias
- moved C3 122.8 mm to (138.4, 69.0)
- moved J2 111.3 mm to (130.3, 114.0)
- moved C4 107.6 mm to (125.5, 127.8), turned to -90 degrees
- moved C8 105.8 mm to (126.0, 104.0), turned to -90 degrees
- moved J1 104.8 mm to (130.2, 72.4)
- moved C5 103.6 mm to (123.5, 109.0), turned to 180 degrees
- moved D1 100.8 mm to (105.5, 71.1), turned to -90 degrees
- moved C10 96.4 mm to (120.0, 108.0), turned to 90 degrees
- moved R2 94.5 mm to (125.5, 118.5), turned to -90 degrees
- moved R1 94.2 mm to (125.5, 114.0), turned to -90 degrees
- moved L1 94.1 mm to (114.5, 79.2)
- moved C9 93.0 mm to (117.0, 108.0), turned to -90 degrees
- moved U1 90.5 mm to (119.0, 104.0)
- moved R8 89.4 mm to (123.0, 104.0), turned to 90 degrees
- moved C13 87.1 mm to (116.3, 92.3), turned to -90 degrees
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- renumbered C7 to C10, C16 to C11, C17 to C12, C18 to C14, C19 to C15, C20 to C16, C21 to C17, C22 to C18, C23 to C28, C24 to C29, C4 to C3, C5 to C4, C3 to C5, C6 to C8, C8 to C9, J12 to J9, R13 to R12, R5 to R8, U5 to U3
Connections:
- net /CAN_module/CAN_L renamed /disp_backlight/LEDB_PWM_DIMM
- net Net-(J15-Pin_2) renamed /display_40_to_22/DISP_SUPPLY_3V3
- BZ1 pad 1: unconnected-(BZ1---Pad1) -> Net-(BZ1--)
- C10 pad 1: +5V -> GNDD
- C10 pad 2: GNDD -> +5V
- C11 pad 1: /disp_backlight/LEDB_ANODE -> +12V
- C12 pad 1: Net-(U4-VCC) -> Net-(U2-VCC)
- C13 pad 1: +3.3V -> GNDD
- C13 pad 2: Net-(J9-Pin_2) -> +3.3V
- C18 pad 1: Net-(J12-Pin_15) -> /camera_15_to_22/CAM0_SUPPLY_3V3
- D1 pad 1: /disp_backlight/LEDB_ANODE -> +12V
- J1 pad 1: Net-(J1-Pin_1) -> +12V
- J10 pad 1: +3.3V -> GNDD
- J10 pad 2: Net-(J10-Pin_2) -> /camera_15_to_22/CAM1_D0_N
- J11 pad 1: +3.3V -> GNDD
- J11 pad 2: Net-(J11-Pin_2) -> /camera_15_to_22/CAM0_D0_N
- J5 pad 10: /GPIO15 -> /RXD1
- J5 pad 11: /GPIO17 -> /RTS1
- J5 pad 12: /GPIO18 -> unconnected-(J5-Pin_12-Pad12)
- J5 pad 13: /GPIO27 -> /BUT1
- J5 pad 15: /GPIO22 -> /BUT6
- J5 pad 16: /GPIO23 -> /INP_BRAKE
- J5 pad 18: /GPIO24 -> /INP_CLUTCH
- J5 pad 19: /GPIO10 -> /BUT4
- J5 pad 21: /GPIO9 -> /BUT3
- J5 pad 22: /GPIO25 -> /LED_AUX
- J5 pad 23: /GPIO11 -> /BUT5
- J5 pad 24: /GPIO8 -> /BUT2
- J5 pad 26: /GPIO7 -> /OBDR_SCLK
- J5 pad 27: /ID_SD -> unconnected-(J5-Pin_27-Pad27)
- J5 pad 28: /ID_SC -> unconnected-(J5-Pin_28-Pad28)
- J5 pad 29: /GPIO5 -> /OBDR_MISO
- J5 pad 3: /GPIO2 -> unconnected-(J5-Pin_3-Pad3)
- J5 pad 31: /GPIO6 -> /OBDR_MOSI
- J5 pad 32: /GPIO12 -> /ACT_PWM
- J5 pad 33: /GPIO13 -> /ACT_DIR
- J5 pad 35: /GPIO19 -> /BUZZER
- J5 pad 36: /GPIO16 -> /CTS1
- J5 pad 37: /GPIO26 -> /BUT7
- J5 pad 38: /GPIO20 -> /LED_WRN
- J5 pad 40: /GPIO21 -> /LED_ALM
- J5 pad 5: /GPIO3 -> /OBDR_INT
- J5 pad 7: /GPIO4 -> /OBDR_CE
- J5 pad 8: /GPIO14 -> /TXD1
- J7 pad 1: +3.3V -> /OBDR_MOSI
- J7 pad 2: Net-(J7-Pin_2) -> /LVL_SHIFT_MISO
- J9 pad 11: unconnected-(J12-Pin_11-Pad11) -> /camera_15_to_22/CAM0_GPIO
- J9 pad 13: unconnected-(J12-Pin_13-Pad13) -> /camera_15_to_22/CAM0_SCL
- J9 pad 14: unconnected-(J12-Pin_14-Pad14) -> /camera_15_to_22/CAM0_SDA
- J9 pad 15: Net-(J12-Pin_15) -> /camera_15_to_22/CAM0_SUPPLY_3V3
- J9 pad 2: unconnected-(J12-Pin_2-Pad2) -> /camera_15_to_22/CAM0_D0_N
- J9 pad 3: unconnected-(J12-Pin_3-Pad3) -> /camera_15_to_22/CAM0_D0_P
- J9 pad 5: unconnected-(J12-Pin_5-Pad5) -> /camera_15_to_22/CAM0_D1_N
- J9 pad 6: unconnected-(J12-Pin_6-Pad6) -> /camera_15_to_22/CAM0_D1_P
- J9 pad 8: unconnected-(J12-Pin_8-Pad8) -> /camera_15_to_22/CAM0_C_N
- J9 pad 9: unconnected-(J12-Pin_9-Pad9) -> /camera_15_to_22/CAM0_C_P
- J9 pad MP: (no net) -> GNDD
- L1 pad 2: /disp_backlight/LEDB_CATHODE -> /DISP_BL_CATH
- R1 pad 1: unconnected-(R1-Pad1) -> /LED_WRN
- R1 pad 2: Net-(J1-Pin_1) -> Net-(J2-Pin_1)
- R10 pad 1: Net-(J11-Pin_2) -> Net-(U2-IADJ)
- R10 pad 2: GNDD -> Net-(R10-Pad2)
- R11 pad 1: Net-(U3-~{RESET}) -> GNDD
- R11 pad 2: unconnected-(R11-Pad2) -> Net-(R10-Pad2)
- R12 pad 1: Net-(U4-FS) -> Net-(U2-FS)
- R2 pad 1: unconnected-(R2-Pad1) -> /LED_ALM
- R2 pad 2: Net-(J2-Pin_1) -> Net-(J3-Pin_1)
- R5 pad 1: Net-(R3-Pad1) -> /INP_CLUTCH
- R6 pad 1: Net-(R4-Pad1) -> /INP_BRAKE
- R7 pad 1: Net-(J8-Pin_2) -> /OBDR_INT
- R7 pad 2: GNDD -> Net-(J7-Pin_6)
- R9 pad 1: Net-(J10-Pin_2) -> /OBDR_INT
- U1 pad 1: (no net) -> /LVL_SHIFT_MISO
- U1 pad 2: (no net) -> GNDD
- U1 pad 3: (no net) -> +3.3V
- U1 pad 4: (no net) -> /OBDR_MISO
- U1 pad 5: (no net) -> GNDD
- U1 pad 6: (no net) -> Net-(U1-OE)
- U1 pad 7: (no net) -> +5V
- U1 pad 8: (no net) -> unconnected-(U1-B1Y-Pad8)
- U2 pad 1: Net-(U2-TXD) -> Net-(U2-VCC)
- U2 pad 3: +5V -> Net-(U2-IADJ)
- U2 pad 4: Net-(U2-RXD) -> GNDD
- U2 pad 5: unconnected-(U2-NC-Pad5) -> Net-(U2-FS)
- U2 pad 7: /CAN_module/CAN_H -> Net-(D1-A)
- U2 pad 8: GNDD -> +12V
- U3 pad 10: unconnected-(U5-T2IN-Pad10) -> /RTS1
- U3 pad 11: unconnected-(U5-T1IN-Pad11) -> /TXD1
- U3 pad 12: unconnected-(U5-R1OUT-Pad12) -> /RXD1
- U3 pad 13: /debug_port/DP_RXD -> /debug_port/DP_TXD
- U3 pad 14: /debug_port/DP_TXD -> /debug_port/DP_RXD
- U3 pad 7: /debug_port/DP_RTS -> /debug_port/DP_CTS
- U3 pad 8: /debug_port/DP_CTS -> /debug_port/DP_RTS
- U3 pad 9: unconnected-(U5-R2OUT-Pad9) -> /CTS1
Routing:
- net GNDD: track 0.00 -> 517.6 mm, vias 0 -> 123
- net +3.3V: track 0.00 -> 195.5 mm, vias 0 -> 9
- net +12V: track 0.00 -> 126.1 mm, vias 0 -> 1
- net /BUT7: track 0.00 -> 73.0 mm, vias 0 -> 3
- net /INP_CLUTCH: track 0.00 -> 70.3 mm, vias 0 -> 5
- net /INP_BRAKE: track 0.00 -> 70.3 mm, vias 0 -> 4
- net +5V: track 0.00 -> 68.1 mm, vias 0 -> 4
- net /BUT5: track 0.00 -> 47.8 mm, vias 0 -> 3
- net /BUT6: track 0.00 -> 45.5 mm, vias 0 -> 2
- net /BUT2: track 0.00 -> 44.4 mm, vias 0 -> 2
- net /display_40_to_22/DISP_SUPPLY_3V3: track 0.00 -> 41.4 mm, vias 0 -> 1
- net /BUT4: track 0.00 -> 39.2 mm, vias 0 -> 1
- net /LED_AUX: track 0.00 -> 38.4 mm, vias 0 -> 4
- net /ACT_DIR: track 0.00 -> 38.2 mm, vias 0 -> 1
- net /BUT3: track 0.00 -> 37.7 mm, vias 0 -> 1
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- added copper zone on B.Cu, net GNDD
- added copper zone on F.Cu, net GNDD
Other:
- board outline added: 64.7 x 89.7 mm
- board text added: "+"
- board text added: "+12V"
- board text added: "+5V"
- board text added: "BRK"
- board text added: "CLH"
- board text added: "CTS"
- board text added: "Connect mounting holes to GND!! Add markings on the top and bottom side to indicate which side's which!!"
- board text added: "DESIGN: M. Nakov DATE: 04.11.2023 VERSION: 1.0"
- board text added: "DIR"
- board text added: "Fix differential pairs!! Thicken power rails!! Give MP a GNDD net!! Fix the thermal relief of U2!!"
- board text added: "GND"
- board text added: "IT"
- board text added: "Make connections between FPCs first!!! Then place biggest components on the top side!!! Signal traces: 8 mil Signal via: 16x32 Power traces: 1 mm (~100 mil) Power traces (12V): 1.2 mm Power via: 0.6x1-2 mm Clearance: 10 mil Try to place all components on the top side!! Otherwise, divide bigger and smaller components on different sides!! Vias should not be on the contacts. Fix this!! Two pins shou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"
- board text added: "PWM"
- board text added: "RTS"
- board text added: "RX"
- board text added: "SCL"
- board text added: "SI"
- board text added: "SO"
- board text added: "SS"
- board text added: "TOP SIDE"
- board text added: "TX"
- board text removed: "Camera Input pin order: L -> R: 15 -> 1"
- board text removed: "Camera Output pin order: L -> R: 1 -> 22"
