File: docs/schematics/aac/Shield.kicad_sch (KiCad schematic)
At the start: 40 parts, among them J1 CONN_LED_ORG, J10 But_4, J11 But_5, J2 CONN_LED_RED, J3 HAT, J4 12V, J5 Actuator, J6 RS232, J7 But_1, J8 But_2, J9 But_3, SW1 SW_Clutch, SW2 SW_Brake, U1 TXU0202

Commit message: Pushing final schematic and PCB.
Parts:
- removed C10, C11, C12, C13, C14, C15: 100n, Capacitor_SMD:C_0805_2012Metric, symbol Device:C
- removed C9: 2.2uF, Capacitor_SMD:C_0805_2012Metric, symbol Device:C
- removed J10: But_4, Connector_PinHeader_2.54mm:PinHeader_1x02_P2.54mm_Vertical, symbol Connector_Generic:Conn_02x01
- removed J11: But_5, Connector_PinHeader_2.54mm:PinHeader_1x02_P2.54mm_Vertical, symbol Connector_Generic:Conn_02x01
- removed J7: But_1, Connector_PinHeader_2.54mm:PinHeader_1x02_P2.54mm_Vertical, symbol Connector_Generic:Conn_02x01
- removed J8: But_2, Connector_PinHeader_2.54mm:PinHeader_1x02_P2.54mm_Vertical, symbol Connector_Generic:Conn_02x01
- removed J9: But_3, Connector_PinHeader_2.54mm:PinHeader_1x02_P2.54mm_Vertical, symbol Connector_Generic:Conn_02x01
- removed R10, R6, R8: 10k, Resistor_SMD:R_0805_2012Metric, symbol Device:R
- added C6, C7: 100n, Capacitor_SMD:C_0805_2012Metric, symbol Device:C
- added J4: CONN_LED_AUX, Connector_PinHeader_2.54mm:PinHeader_2x01_P2.54mm_Horizontal, symbol Connector_Generic:Conn_02x01
- added J7: CAN_Module, Connector_PinHeader_2.54mm:PinHeader_1x07_P2.54mm_Vertical, symbol Connector_Generic:Conn_01x07
- added R3, R4: 140, Resistor_SMD:R_0805_2012Metric, symbol Device:R
- J1: renamed from J4; footprint (none) -> Connector_PinHeader_2.54mm:PinHeader_1x02_P2.54mm_Horizontal
- J2: renamed from J1; footprint Connector_PinHeader_2.54mm:PinHeader_1x02_P2.54mm_Vertical -> Connector_PinHeader_2.54mm:PinHeader_2x01_P2.54mm_Horizontal
- J3: renamed from J2; footprint Connector_PinHeader_2.54mm:PinHeader_1x02_P2.54mm_Vertical -> Connector_PinHeader_2.54mm:PinHeader_2x01_P2.54mm_Horizontal
- J6: renamed from J5; footprint Connector_PinHeader_2.54mm:PinHeader_2x05_P2.54mm_Vertical -> Connector_PinHeader_2.54mm:PinHeader_2x03_P2.54mm_Vertical; symbol Connector_Generic:Conn_02x05_Odd_Even -> Connector_Generic:Conn_02x03_Odd_Even
- J8: renamed from J6; footprint Connector_PinHeader_2.54mm:PinHeader_1x07_P2.54mm_Horizontal -> Connector_PinHeader_2.54mm:PinHeader_1x06_P2.54mm_Horizontal
- R5: renamed from R3; value 10k -> 10K
- R6: renamed from R4; value 10k -> 10K
- R7, R9: value 10k -> 1K
- SW1, SW2: footprint (none) -> Connector_PinHeader_2.54mm:PinHeader_2x01_P2.54mm_Horizontal
- renumbered C7 to C10, C4 to C3, C5 to C4, C3 to C5, C6 to C8, C8 to C9, J3 to J5, R5 to R8
Connections:
- net GPIO20 is gone; now on net LED_WRN: J5.38 (Pin_38)
- net GPIO21 is gone; now on net LED_ALM: J5.40 (Pin_40)
- net GPIO23 is gone; now on net INP_BRAKE: J5.16 (Pin_16)
- net GPIO24 is gone; now on net INP_CLUTCH: J5.18 (Pin_18)
- net GPIO3 is gone; now on net OBDR_INT: J5.5 (Pin_5)
- net +12V: no longer J6.3 (Pin_3), J6.7 (Pin_7), J6.9 (Pin_9)
- net +3.3V: now also U1.3 (VCCa), C6.1, C7.1; no longer U1. (VCCb)
- net +5V: now also C10.2, U1.7 (VCCb), J7.5 (Pin_5); no longer C10.1, U1. (VCCb)
- net GNDD: now also C10.1, U1.2 (GND), U1.5 (A1), J4.2 (Pin_2), J7.7 (Pin_7); no longer C10.2, J6.10 (Pin_10), J6.4 (Pin_4), J6.8 (Pin_8), R7.2, U1. (VCCb)
- net at R8.1: now also U1.6 (OE); no longer U1. (VCCb)
- net OBDR_INT: now reaches R7.1
- net OBDR_INT: now also R9.1
- net at BZ1.1 (-): now also R4.2
- net INP_BRAKE: now reaches R6.1, SW2.1
- net INP_BRAKE: now also J6.2 (Pin_2), C7.2
- net INP_CLUTCH: now reaches J6.1 (Pin_1)
- net INP_CLUTCH: now also R5.1, SW1.1, C6.2
- net LED_ALM: now reaches R2.1
- net LED_WRN: now reaches R1.1
- removed net CAN_module/MOD_SO: U1. (VCCb)
- net GPIO10 renamed BUT4
- net GPIO11 renamed BUT5
- net GPIO12 renamed ACT_PWM
- net ACT_PWM: now also J6.3 (Pin_3)
- net GPIO13 renamed ACT_DIR
- net ACT_DIR: now also J6.4 (Pin_4)
- net GPIO14 renamed TXD1
- net GPIO15 renamed RXD1
- net GPIO16 renamed CTS1
- net GPIO17 renamed RTS1
- net GPIO18: no longer names the net of J5.12 (Pin_12)
- net GPIO19 renamed BUZZER
- net BUZZER: now also R4.1
- net GPIO2: no longer names the net of J5.3 (Pin_3)
- net GPIO22 renamed BUT6
- net GPIO25 renamed LED_AUX
- net LED_AUX: now also R3.1
- net GPIO26 renamed BUT7
- net GPIO27 renamed BUT1
- net GPIO4 renamed OBDR_CE
- net OBDR_CE: now also J7.3 (Pin_3)
- net GPIO5 renamed OBDR_MISO
- net OBDR_MISO: now also U1.4 (A2Y)
- net GPIO6 renamed OBDR_MOSI
- net OBDR_MOSI: now also J7.1 (Pin_1)
- net GPIO7 renamed OBDR_SCLK
- net OBDR_SCLK: now also J7.4 (Pin_4)
- net GPIO8 renamed BUT2
- net GPIO9 renamed BUT3
- net ID_SC: no longer names the net of J5.28 (Pin_28)
- net ID_SD: no longer names the net of J5.27 (Pin_27)
- new net: J4.1 (Pin_1), R3.2
- new net: J7.6 (Pin_6), R7.2
- new net LVL_SHIFT_MISO: J7.2 (Pin_2), U1.1 (B2)
- no-connect marks 10 -> 6
Other:
- removed sheet CAN_module
- added sheet control_buttons (control_btns.kicad_sch)
- sheet debug_port ports: added IN_CTS, IN_RTS, IN_RX, IN_TX; removed none
- sheet display_40_to_22 ports: added BL_AN, BL_CATH; removed none
- note added: "GND"
- note added: "GPIO10"
- note added: "GPIO11"
- note added: "GPIO12"
- note added: "GPIO13"
- note added: "GPIO14"
- note added: "GPIO15"
- note added: "GPIO16"
- note added: "GPIO17"
- note added: "GPIO18"
- note added: "GPIO19"
- note added: "GPIO2"
- note added: "GPIO20"
- note added: "GPIO21"
- note added: "GPIO22"
- note added: "GPIO23"
- note added: "GPIO24"
- note added: "GPIO25"
- note added: "GPIO26"
- note added: "GPIO27"
- note added: "GPIO3"
- note added: "GPIO4"
- note added: "GPIO5"
- note added: "GPIO6"
- note added: "GPIO7"
- note added: "GPIO8"
- note added: "GPIO9"
- note added: "ID_SC"
- note added: "ID_SD"
- note added: "INT"
- note added: "MOD_MISO"
- note added: "MOD_MOSI"
- note added: "MOD_SCLK"
- note added: "MOD_SS"
- note added: "Pins on the right hand side should be flipped!!"
- note added: "VCC (+5V)"
- company: (none) -> Robert Bosch GmbH
- title: (none) -> DA_Shield_Schematic
- moved on the sheet: BZ1, C10, C2, C3, C4, C5, J1, J8, R5, R6, SW1, SW2
