File: docs/schematics/aac/camera_map.kicad_sch (KiCad schematic)
At the start: 3 parts

Commit message: Pushing final schematic and PCB.
Parts:
- added C19: 100n, Capacitor_SMD:C_0805_2012Metric, symbol Device:C
- added J?: Berry_CAM1, Connector_FFC-FPC:Hirose_FH12-22S-0.5SH_1x22-1MP_P0.50mm_Horizontal, symbol Connector_Generic:Conn_01x22
- added J?: Camera, Connector_FFC-FPC:TE_1-84952-5_1x15-1MP_P1.0mm_Horizontal, symbol Connector_Generic:Conn_01x15
- J?: value Berry_CAM -> Berry_CAM0; footprint (none) -> Connector_FFC-FPC:Hirose_FH12-22S-0.5SH_1x22-1MP_P0.50mm_Horizontal
- renumbered C22 to C18
Connections:
- net GNDD: now also C19.2, J?.1 (Pin_1), J?.1 (Pin_1), J?.10 (Pin_10), J?.10 (Pin_10), J?.13 (Pin_13), J?.16 (Pin_16), J?.19 (Pin_19), J?.4 (Pin_4), J?.4 (Pin_4), J?.7 (Pin_7), J?.7 (Pin_7)
- net CAM0_GPIO: now reaches J?.17 (Pin_17)
- net CAM0_GPIO: now also J?.11 (Pin_11)
- net CAM0_D0_N: now reaches J?.2 (Pin_2)
- net CAM0_D0_N: now also J?.2 (Pin_2)
- net CAM0_SCL: now reaches J?.20 (Pin_20)
- net CAM0_SCL: now also J?.13 (Pin_13)
- net CAM0_SDA: now reaches J?.21 (Pin_21)
- net CAM0_SDA: now also J?.14 (Pin_14)
- net CAM0_SUPPLY_3V3: now reaches J?.22 (Pin_22)
- net CAM0_SUPPLY_3V3: now also C18.1, J?.15 (Pin_15)
- net CAM0_D0_P: now reaches J?.3 (Pin_3)
- net CAM0_D0_P: now also J?.3 (Pin_3)
- net CAM0_D1_N: now reaches J?.5 (Pin_5)
- net CAM0_D1_N: now also J?.5 (Pin_5)
- net CAM0_D1_P: now reaches J?.6 (Pin_6)
- net CAM0_D1_P: now also J?.6 (Pin_6)
- net CAM0_C_N: now reaches J?.8 (Pin_8)
- net CAM0_C_N: now also J?.8 (Pin_8)
- net CAM0_C_P: now reaches J?.9 (Pin_9)
- net CAM0_C_P: now also J?.9 (Pin_9)
- new net CAM1_C_N: J?.8 (Pin_8), J?.8 (Pin_8)
- new net CAM1_C_P: J?.9 (Pin_9), J?.9 (Pin_9)
- new net CAM1_D0_N: J?.2 (Pin_2), J?.2 (Pin_2)
- new net CAM1_D0_P: J?.3 (Pin_3), J?.3 (Pin_3)
- new net CAM1_D1_N: J?.5 (Pin_5), J?.5 (Pin_5)
- new net CAM1_D1_P: J?.6 (Pin_6), J?.6 (Pin_6)
- new net CAM1_GPIO: J?.11 (Pin_11), J?.17 (Pin_17)
- new net CAM1_SCL: J?.13 (Pin_13), J?.20 (Pin_20)
- new net CAM1_SDA: J?.14 (Pin_14), J?.21 (Pin_21)
- new net CAM1_SUPPLY_3V3: C19.1, J?.15 (Pin_15), J?.22 (Pin_22)
- no-connect marks 5 -> 12
Other:
- moved on the sheet: C18, J?
