File: docs/schematics/aac/debug_port.kicad_sch (KiCad schematic)
At the start: 5 parts

Commit message: Pushing final schematic and PCB.
Parts:
- added C?: 2.2uF, Capacitor_SMD:C_0805_2012Metric, symbol Device:C
Connections:
- net DP_CTS: now also U?.7 (T2OUT); no longer U?.8 (R2IN)
- net DP_RTS: now also U?.8 (R2IN); no longer U?.7 (T2OUT)
- net DP_RXD: now also U?.14 (T1OUT); no longer U?.13 (R1IN)
- net DP_TXD: now also U?.13 (R1IN); no longer U?.14 (T1OUT)
- net DP_VCC: now also C?.2
- net GNDD: now also C?.1
- net IN_RTS: now reaches U?.10 (T2IN)
- net IN_TX: now reaches U?.11 (T1IN)
- net IN_RX: now reaches U?.12 (R1OUT)
- net IN_CTS: now reaches U?.9 (R2OUT)
Changed lines of the file:
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@@
 (kicad_sch (version 20230121) (generator eeschema)
   (paper "A4")
+  (junction (at 128.27 69.85) (diameter 0) (color 0 0 0 0)
+  )
+  (wire (pts (xy 153.67 125.73) (xy 161.29 125.73))
+    (stroke (width 0) (type default))
+  )
+  (wire (pts (xy 151.13 128.27) (xy 161.29 128.27))
+    (stroke (width 0) (type default))
+  )
   (wire (pts (xy 170.18 99.06) (xy 170.18 106.045))
     (stroke (width 0) (type default))
   )
-  (wire (pts (xy 153.67 125.73) (xy 161.29 125.73))
-    (stroke (width 0) (type default))
-  )
   (wire (pts (xy 128.27 69.85) (xy 128.27 78.74))
     (stroke (width 0) (type default))
@@
     (stroke (width 0) (type default))
   )
+  (wire (pts (xy 148.59 130.81) (xy 161.29 130.81))
+    (stroke (width 0) (type default))
+  )
   (wire (pts (xy 151.13 121.92) (xy 151.13 128.27))
     (stroke (width 0) (type default))
@@
     (stroke (width 0) (type default))
   )
-  (wire (pts (xy 148.59 130.81) (xy 161.29 130.81))
-    (stroke (width 0) (type default))
-  )
   (wire (pts (xy 148.59 86.36) (xy 154.94 86.36))
     (stroke (width 0) (type default))
@@
     (stroke (width 0) (type default))
   )
+  (wire (pts (xy 125.73 69.85) (xy 128.27 69.85))
+    (stroke (width 0) (type default))
+  )
   (wire (pts (xy 148.59 99.06) (xy 170.18 99.06))
     (stroke (width 0) (type default))
@@
     (stroke (width 0) (type default))
   )
+  (wire (pts (xy 154.94 123.19) (xy 161.29 123.19))
+    (stroke (width 0) (type default))
+  )
+  (wire (pts (xy 115.57 69.85) (xy 118.11 69.85))
+    (stroke (width 0) (type default))
+  )
   (wire (pts (xy 128.27 69.85) (xy 138.43 69.85))
     (stroke (width 0) (type default))
   )
-  (wire (pts (xy 154.94 123.19) (xy 161.29 123.19))
-    (stroke (width 0) (type default))
-  )
-  (wire (pts (xy 151.13 128.27) (xy 161.29 128.27))
-    (stroke (width 0) (type default))
-  )
   (wire (pts (xy 148.59 127) (xy 148.59 130.81))
     (stroke (width 0) (type default))
@@
     (stroke (width 0) (type default))
   )
-  (hierarchical_label "DP_CTS" (shape output) (at 161.29 130.81 0) (fields_autoplaced)
-    (effects (font (size 1.27 1.27)) (justify left))
+  (wire (pts (xy 115.57 69.85) (xy 115.57 72.39))
+    (stroke (width 0) (type default))
+  )
+  (hierarchical_label "DP_CTS" (shape output) (at 161.29 125.73 0) (fields_autoplaced)
+    (effects (font (size 1.27 1.27)) (justify left))
+  )
+  (hierarchical_label "IN_RX" (shape input) (at 107.95 121.92 180) (fields_autoplaced)
+    (effects (font (size 1.27 1.27)) (justify right))
+  )
+  (hierarchical_label "IN_CTS" (shape input) (at 107.95 127 180) (fields_autoplaced)
+    (effects (font (size 1.27 1.27)) (justify right))
   )
   (hierarchical_label "DP_VCC" (shape input) (at 138.43 69.85 0) (fields_autoplaced)
     (effects (font (size 1.27 1.27)) (justify left))
   )
-  (hierarchical_label "DP_RXD" (shape input) (at 161.29 128.27 0) (fields_autoplaced)
-    (effects (font (size 1.27 1.27)) (justify left))
-  )
-  (hierarchical_label "DP_TXD" (shape output) (at 161.29 123.19 0) (fields_autoplaced)
-    (effects (font (size 1.27 1.27)) (justify left))
-  )
-  (hierarchical_label "DP_RTS" (shape output) (at 161.29 125.73 0) (fields_autoplaced)
-    (effects (font (size 1.27 1.27)) (justify left))
-  )
-  (netclass_flag "" (length 2.54) (shape round) (at 107.95 116.84 90)
-    (effects (font (size 1.27 1.27)) (justify left bottom))
-    (property "Netclass" "RTS1" (at 99.695 116.84 0)
-      (effects (font (size 1.27 1.27) italic) (justify left))
-    )
-  )
-  (netclass_flag "" (length 2.54) (shape round) (at 107.95 121.92 90)
-    (effects (font (size 1.27 1.27)) (justify left bottom))
-    (property "Netclass" "RXD1" (at 99.06 121.92 0)
-      (effects (font (size 1.27 1.27) italic) (justify left))
-    )
-  )
-  (netclass_flag "" (length 2.54) (shape round) (at 107.95 111.76 90)
-    (effects (font (size 1.27 1.27)) (justify left bottom))
-    (property "Netclass" "TXD1" (at 99.695 111.76 0)
-      (effects (font (size 1.27 1.27) italic) (justify left))
-    )
-  )
-  (netclass_flag "" (length 2.54) (shape round) (at 107.95 127 90)
-    (effects (font (size 1.27 1.27)) (justify left bottom))
-    (property "Netclass" "CTS1" (at 99.695 127 0)
-      (effects (font (size 1.27 1.27) italic) (justify left))
-    )
+  (hierarchical_label "DP_RXD" (shape output) (at 161.29 123.19 0) (fields_autoplaced)
+    (effects (font (size 1.27 1.27)) (justify left))
+  )
+  (hierarchical_label "DP_TXD" (shape output) (at 161.29 128.27 0) (fields_autoplaced)
+    (effects (font (size 1.27 1.27)) (justify left))
+  )
+  (hierarchical_label "IN_RTS" (shape input) (at 107.95 116.84 180) (fields_autoplaced)
+    (effects (font (size 1.27 1.27)) (justify right))
+  )
+  (hierarchical_label "IN_TX" (shape input) (at 107.95 111.76 180) (fields_autoplaced)
+    (effects (font (size 1.27 1.27)) (justify right))
+  )
+  (hierarchical_label "DP_RTS" (shape output) (at 161.29 130.81 0) (fields_autoplaced)
+    (effects (font (size 1.27 1.27)) (justify left))
   )
   (symbol (lib_id "power:GNDD") (at 128.27 139.7 0) (unit 1)
@@
         )
         (path "/c8a79654-8f73-41b9-af0f-6eb1ff86e46c/a63436a7-3aaf-4681-9078-7b8c94da3f0e"
-          (reference "#PWR048") (unit 1)
+          (reference "#PWR042") (unit 1)
         )
       )
@@
         )
         (path "/c8a79654-8f73-41b9-af0f-6eb1ff86e46c/a63436a7-3aaf-4681-9078-7b8c94da3f0e"
-          (reference "C20") (unit 1)
+          (reference "C16") (unit 1)
         )
       )
@@
         )
         (path "/c8a79654-8f73-41b9-af0f-6eb1ff86e46c/a63436a7-3aaf-4681-9078-7b8c94da3f0e"
-          (reference "C19") (unit 1)
+          (reference "C15") (unit 1)
         )
       )
@@
         )
         (path "/c8a79654-8f73-41b9-af0f-6eb1ff86e46c/a63436a7-3aaf-4681-9078-7b8c94da3f0e"
-          (reference "#PWR046") (unit 1)
+          (reference "#PWR040") (unit 1)
+        )
+      )
+    )
+  )
+  (symbol (lib_id "Device:C") (at 121.92 69.85 90) (mirror x) (unit 1)
+    (in_bom yes) (on_board yes) (dnp no)
+    (property "Reference" "C?" (at 124.46 73.66 90)
+      (effects (font (size 1.27 1.27)) (justify left))
+    )
+    (property "Value" "2.2uF" (at 125.095 76.2 90)
+      (effects (font (size 1.27 1.27)) (justify left))
+    )
+    (property "Footprint" "Capacitor_SMD:C_0805_2012Metric" (at 125.73 70.8152 0)
+      (effects (font (size 1.27 1.27)) hide)
+    )
+    (property "Datasheet" "~" (at 121.92 69.85 0)
+      (effects (font (size 1.27 1.27)) hide)
+    )
+    (pin "1")
+    (pin "2")
+    (instances
+      (project "Shield"
+        (path "/c8a79654-8f73-41b9-af0f-6eb1ff86e46c"
+          (reference "C?") (unit 1)
+        )
+        (path "/c8a79654-8f73-41b9-af0f-6eb1ff86e46c/a63436a7-3aaf-4681-9078-7b8c94da3f0e"
+          (reference "C13") (unit 1)
         )
       )
@@
         )
         (path "/c8a79654-8f73-41b9-af0f-6eb1ff86e46c/a63436a7-3aaf-4681-9078-7b8c94da3f0e"
-          (reference "C21") (unit 1)
+          (reference "C17") (unit 1)
+        )
+      )
+    )
+  )
+  (symbol (lib_id "power:GNDD") (at 115.57 72.39 0) (unit 1)
+    (in_bom yes) (on_board yes) (dnp no) (fields_autoplaced)
+    (property "Reference" "#PWR?" (at 115.57 78.74 0)
+      (effects (font (size 1.27 1.27)) hide)
+    )
+    (property "Value" "GNDD" (at 115.57 76.2 0)
+      (effects (font (size 1.27 1.27)) hide)
+    )
+    (property "Footprint" "" (at 115.57 72.39 0)
+      (effects (font (size 1.27 1.27)) hide)
+    )
+    (property "Datasheet" "" (at 115.57 72.39 0)
+      (effects (font (size 1.27 1.27)) hide)
+    )
+    (pin "1")
+    (instances
+      (project "Shield"
+        (path "/c8a79654-8f73-41b9-af0f-6eb1ff86e46c"
+          (reference "#PWR?") (unit 1)
+        )
+        (path "/c8a79654-8f73-41b9-af0f-6eb1ff86e46c/a63436a7-3aaf-4681-9078-7b8c94da3f0e"
+          (reference "#PWR039") (unit 1)
         )
       )
@@
         )
         (path "/c8a79654-8f73-41b9-af0f-6eb1ff86e46c/a63436a7-3aaf-4681-9078-7b8c94da3f0e"
-          (reference "U5") (unit 1)
+          (reference "U3") (unit 1)
         )
       )
@@
         )
         (path "/c8a79654-8f73-41b9-af0f-6eb1ff86e46c/a63436a7-3aaf-4681-9078-7b8c94da3f0e"
-          (reference "C18") (unit 1)
+          (reference "C14") (unit 1)
         )
       )
@@
         )
         (path "/c8a79654-8f73-41b9-af0f-6eb1ff86e46c/a63436a7-3aaf-4681-9078-7b8c94da3f0e"
-          (reference "#PWR047") (unit 1)
-        )
-      )
+          (reference "#PWR041") (unit 1)
+        )
+      )
