File: docs/schematics/aac/disp_backlight.kicad_sch (KiCad schematic)
At the start: 7 parts, among them U4 TPS92511DDA

Commit message: Pushing final schematic and PCB.
Parts:
- removed R12: 5.1K, Resistor_SMD:R_0805_2012Metric, symbol Device:R
- added R10: 5.1K, Resistor_SMD:R_0805_2012Metric, symbol Device:R
- added R11: PT15LV 25K, Potentiometer_THT:Potentiometer_ACP_CA14V-15_Vertical, symbol Device:R_Trim
- L1: value 47 uH -> 330 uH; footprint Inductor_SMD:L_7.3x7.3_H4.5 -> Inductor_SMD:L_SigTra_SC3316F
- U2: renamed from U4; footprint TPS92511DDA:VREG_LM5017MR_NOPB -> Package_SO:SOIC-8-1EP_3.9x4.9mm_P1.27mm_EP2.29x3mm_ThermalVias
- renumbered C16 to C11, C17 to C12, R13 to R12
Connections:
- net GNDD: now also U2.9 (HD), R11.1
- net LEDB_ANODE: now also U2.8 (VIN); no longer U2.5 (VIN)
- net LEDB_PWM_DIMM: now also U2.6 (DIM); no longer U2.7 (DIM)
- net at D1.2 (A), L1.1: now also U2.7 (LX); no longer U2.6 (LX)
- net at U2.3 (IADJ): now also R10.1
- net at R12.1: now also U2.5 (FS); no longer U2.8 (FS)
- new net: R10.2, R11.2
Other:
- note added: "ADD A POTENTIOMETER ON IADJ!!! (min 50 mA, max 300 mA) Lmin = 330 uH Radj E [5; 30] kOhm"
- note added: "L = ((12 - 9.6) * 9.6) / (2 * 0.29 * 12 * 100 * 10^3) L = 0.00003310344 ~ 3.31 * 10^(-5) = 33.1 uH => 47 uH Fix the footprint of the TPS!!"
- note removed: "L = ((12 - 9.6) * 9.6) / (2 * 0.29 * 12 * 100 * 10^3) L = 0.00003310344 ~ 3.31 * 10^(-5) = 33.1 uH => 47 uH Turn resistors upside down!! Check the values of the filtering capacitors!!"
- moved on the sheet: D1, R12
