File: docs/schematics/aac/display_mapping.kicad_sch (KiCad schematic)
At the start: 7 parts

Commit message: Pushing final schematic and PCB.
Parts:
- J?: footprint (none) -> Connector_FFC-FPC:Hirose_FH12-40S-0.5SH_1x40-1MP_P0.50mm_Horizontal
- J?: footprint (none) -> Connector_FFC-FPC:Hirose_FH12-22S-0.5SH_1x22-1MP_P0.50mm_Horizontal
- JP? (x2): footprint (none) -> Jumper:SolderJumper-2_P1.3mm_Open_RoundedPad1.0x1.5mm
- R?: value 10k -> 10K
Connections:
- net D1N: now reaches J?.11 (Pin_11)
- net D1N: now also J?.5 (Pin_5)
- net D1P: now reaches J?.12 (Pin_12)
- net D1P: now also J?.6 (Pin_6)
- net D2N: now reaches J?.14 (Pin_14)
- net D2N: now also J?.11 (Pin_11)
- net D2P: now reaches J?.15 (Pin_15)
- net D2P: now also J?.12 (Pin_12)
- net DCLKN: now reaches J?.17 (Pin_17)
- net DCLKN: now also J?.8 (Pin_8)
- net DCLKP: now reaches J?.18 (Pin_18)
- net DCLKP: now also J?.9 (Pin_9)
- net DISP_SUPPLY_3V3: now reaches C?.1, J?.2 (Pin_2), J?.3 (Pin_3), R?.1
- net DISP_SUPPLY_3V3: now also J?.22 (Pin_22), JP?.1 (A)
- net D3N: now reaches J?.20 (Pin_20)
- net D3N: now also J?.14 (Pin_14)
- net D3P: now reaches J?.21 (Pin_21)
- net D3P: now also J?.15 (Pin_15)
- net BL_CATH: now reaches J?.31 (Pin_31), J?.32 (Pin_32)
- net BL_AN: now reaches J?.39 (Pin_39), J?.40 (Pin_40)
- net D0N: now reaches J?.8 (Pin_8)
- net D0N: now also J?.2 (Pin_2)
- net D0P: now reaches J?.9 (Pin_9)
- net D0P: now also J?.3 (Pin_3)
Other:
- note added: "Change SUPPLY_3V3 to DISP_SUPPLY_3V3!! Add comments to the jumpers about what they influence!!!"
- note added: "L/R"
- note added: "Up / Down"
